File: swervepcb.kicad_pcb (KiCad board)
At the start: 2 copper layers, 73 parts, among them J1 RJ45_LED, U1 Teensy4.1, U10 PCB_Mounted_XT30, U11 BAT, U12 L298P, U13 L298P, U14 L7805, U15 L7805, U16 PCB_Mounted_XT30, U17 PCB_Mounted_XT30, U18 PCB_Mounted_XT30, U2 NRF24L01_Breakout, U3 L298P, U4 L298P, U5 L7805, U6 L7805, U7 PCB_Mounted_XT30, U8 PCB_Mounted_XT30, U9 PCB_Mounted_XT30

Commit message: finalized motor controller design
Parts:
- added U19: PCB_Mounted_XT30, teensy:RightAngleXT30-M, F.Cu at (206.4, 46.8)
- C1: footprint L298P:L298P -> Capacitor_THT:CP_Radial_D8.0mm_P3.50mm
- moved U8 202.4 mm to (223.0, 74.6)
- moved R1 186.3 mm to (207.5, 110.0), turned to 90 degrees
- moved D9 152.5 mm to (212.2, 105.6), turned to -90 degrees
- moved C1 126.1 mm to (201.9, 110.8), turned to 90 degrees
- moved D15 81.4 mm to (229.2, 82.5), turned to 180 degrees
- moved C3 77.6 mm to (208.0, 74.5), turned to -90 degrees
- moved D16 73.8 mm to (221.6, 86.5)
- moved U18 69.1 mm to (167.5, 145.3), turned to 0 degrees
- moved D11 66.2 mm to (229.2, 90.5), turned to 180 degrees
- moved D12 56.2 mm to (221.6, 94.5)
- moved U7 46.2 mm to (192.9, 74.6), turned to 0 degrees
- moved U5 40.8 mm to (214.6, 113.2), turned to -90 degrees
- moved D6 39.7 mm to (194.3, 90.5), turned to 180 degrees
- moved U9 21.8 mm to (49.2, 61.1)
- moved D1 21.4 mm to (186.7, 86.5)
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Connections:
- U10 pad 1: (no net) -> Net-(D17-Pad2)
- U10 pad 2: (no net) -> Net-(D13-Pad2)
- U16 pad 1: (no net) -> Net-(D23-Pad2)
- U16 pad 2: (no net) -> Net-(D19-Pad2)
- U17 pad 1: (no net) -> Net-(D33-Pad2)
- U17 pad 2: (no net) -> Net-(D29-Pad2)
- U18 pad 1: (no net) -> Net-(D25-Pad2)
- U18 pad 2: (no net) -> Net-(D21-Pad2)
- U7 pad 1: (no net) -> Net-(D5-Pad2)
- U7 pad 2: (no net) -> Net-(D1-Pad2)
- U8 pad 1: (no net) -> Net-(D15-Pad2)
- U8 pad 2: (no net) -> Net-(D11-Pad2)
- U9 pad 1: (no net) -> Net-(D7-Pad2)
- U9 pad 2: (no net) -> Net-(D3-Pad2)
Routing:
- net GND: track 76.7 -> 224.2 mm, vias 0 -> 5
- net +5V: track 0.00 -> 95.9 mm
- net M1 IN1: track 0.00 -> 34.6 mm, vias 0 -> 2
- net Net-(C1-Pad2): track 0.00 -> 32.3 mm
- net M1 PWM1: track 0.00 -> 31.5 mm, vias 0 -> 2
- net M1 IN2: track 0.00 -> 29.0 mm, vias 0 -> 2
- net Net-(D11-Pad2): track 0.00 -> 26.5 mm
- net Net-(D5-Pad2): track 0.00 -> 26.5 mm
- net Net-(F1-Pad2): track 0.00 -> 20.7 mm
- net Net-(D15-Pad2): track 0.00 -> 17.3 mm
- net Net-(D1-Pad2): track 0.00 -> 17.3 mm
- net M1 IN4: track 0.00 -> 10.9 mm
- net M1 PWM2: track 0.00 -> 10.7 mm
- net M1 IN3: track 0.00 -> 10.5 mm
- net Net-(D9-Pad2): track 0.00 -> 5.14 mm
- added copper zone on F.Cu, net +5V
- added copper zone on B.Cu, net GND

Commit message: progress
Parts:
- removed the C2 at (124.9, 49.7)
- removed the D3 at (120.0, 34.3)
- removed D33, D34, D35, D36: , Diode_THT:D_DO-41_SOD81_P7.62mm_Horizontal
- removed the D4 at (59.5, 96.0)
- removed the D7 at (80.3, 76.5)
- removed the D8 at (82.2, 80.7)
- removed F5: 2a, Fuse:Fuseholder_Cylinder-5x20mm_Schurter_0031_8201_Horizontal_Open
- removed the U1 at (46.7, 23.5)
- removed U10, U16, U17, U18, U19, U9: PCB_Mounted_XT30, teensy:RightAngleXT30-M
- removed U12, U13: L298P, L298P:L298P
- removed U14, U15: L7805, L7805CV:STMicroelectronics-TO-220-3-0-0-0
- added C3: 220uF, Capacitor_THT:CP_Radial_D8.0mm_P3.50mm, F.Cu at (303.8, 106.8)
- added D11: , Diode_THT:D_DO-41_SOD81_P7.62mm_Horizontal, F.Cu at (233.6, 135.1)
- added D12: , Diode_THT:D_DO-41_SOD81_P7.62mm_Horizontal, F.Cu at (304.8, 90.3)
- added D15: , Diode_THT:D_DO-41_SOD81_P7.62mm_Horizontal, F.Cu at (273.5, 120.8)
- added D16: , Diode_THT:D_DO-41_SOD81_P7.62mm_Horizontal, F.Cu at (306.7, 81.8)
- added F3: 2a, Fuse:Fuseholder_Cylinder-5x20mm_Schurter_0031_8201_Horizontal_Open, F.Cu at (129.0, 176.2)
- added LED1: PWR-LED, LED_THT:LED_D5.0mm, F.Cu at (42.5, 57.2)
- added LED2: PWR-LED, LED_THT:LED_D5.0mm, F.Cu at (315.1, 97.2)
- added LED3: PWR-LED, LED_THT:LED_D5.0mm, F.Cu at (300.3, 115.3)
- added LED4: PWR-LED, LED_THT:LED_D5.0mm, F.Cu at (312.7, 105.8)
- added M2O1: PCB_Mounted_XT30, teensy:RightAngleXT30-M, F.Cu at (298.2, 83.3)
- added M2O2: PCB_Mounted_XT30, teensy:RightAngleXT30-M, F.Cu at (253.6, 128.5)
- added M3O1: PCB_Mounted_XT30, teensy:RightAngleXT30-M, F.Cu at (258.7, 117.3)
- added M3O2: PCB_Mounted_XT30, teensy:RightAngleXT30-M, F.Cu at (240.3, 128.5)
- added M4O2: PCB_Mounted_XT30, teensy:RightAngleXT30-M, F.Cu at (227.0, 128.5)
- added U3: L298P, L298P:L298P, F.Cu at (184.5, 83.0)
- added U7: Teensy4.1, teensy:Teensy41, F.Cu at (48.8, 106.5)
- C8: footprint Diode_THT:D_DO-41_SOD81_P7.62mm_Horizontal -> Capacitor_THT:CP_Radial_D8.0mm_P3.50mm
- D10, D27, D28, D9: value PWR-LED -> (none); footprint LED_THT:LED_D5.0mm -> Diode_THT:D_DO-41_SOD81_P7.62mm_Horizontal
- F0: renamed from F3; value 10a -> 8a
- R1, R2, R3, R4: footprint Resistor_SMD:R_0805_2012Metric_Pad1.20x1.40mm_HandSolder -> Resistor_THT:R_Axial_DIN0309_L9.0mm_D3.2mm_P12.70mm_Horizontal
- U2: value NRF24L01_Breakout -> L298P; footprint RF_Module:nRF24L01_Breakout -> L298P:L298P
- U6: value L7805 -> NRF24L01_Breakout; footprint L7805CV:STMicroelectronics-TO-220-3-0-0-0 -> RF_Module:nRF24L01_Breakout
- moved C8 275.8 mm to (291.3, 115.3)
- moved D22 247.2 mm to (306.7, 86.0)
- moved C9 230.1 mm to (267.2, 112.3)
- moved D25 219.6 mm to (289.9, 108.4)
- moved R3 213.2 mm to (239.0, 111.3)
- moved C7 211.8 mm to (306.1, 97.2)
- moved C5 210.3 mm to (319.4, 88.7)
- moved D24 208.7 mm to (291.0, 104.2)
- moved D32 207.6 mm to (318.1, 81.8)
- moved R4 206.6 mm to (221.9, 122.5)
- moved C4 205.3 mm to (286.2, 124.9)
- moved D26 197.0 mm to (256.3, 135.1)
- moved D13 195.1 mm to (291.0, 99.9)
- moved R2 185.6 mm to (237.7, 122.5)
- moved D21 184.6 mm to (273.5, 125.1)
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- renumbered C3 to C2, D5 to D3, D6 to D4, D11 to D5, D12 to D6, D15 to D7, D16 to D8, U7 to M1O1, U8 to M1O2, U11 to U0, U3 to U1
Connections:
- C1 pad 2: Net-(C1-Pad2) -> Net-(C2-Pad1)
- C2 pad 1: +5V -> Net-(C2-Pad1)
- C4 pad 1: +5V -> Net-(U2-Pad6)
- C5 pad 2: Net-(C5-Pad2) -> Net-(LED3-Pad1)
- C6 pad 1: +5V -> Net-(LED3-Pad1)
- C6 pad 2: Net-(C6-Pad2) -> GND
- C7 pad 2: GND -> Net-(LED4-Pad1)
- C8 pad 1: +5V -> Net-(LED4-Pad1)
- D1 pad 1: +5V -> Net-(C2-Pad1)
- D10 pad 1: Net-(C2-Pad2) -> Net-(U2-Pad4)
- D10 pad 2: Net-(D10-Pad2) -> GND
- D13 pad 1: +5V -> Net-(U2-Pad6)
- D13 pad 2: Net-(D13-Pad2) -> Net-(U2-Pad16)
- D14 pad 1: Net-(D13-Pad2) -> Net-(U2-Pad16)
- D17 pad 1: +5V -> Net-(LED3-Pad1)
- D17 pad 2: Net-(D17-Pad2) -> Net-(M3O1-Pad2)
- D18 pad 1: Net-(D17-Pad2) -> Net-(M3O1-Pad2)
- D19 pad 1: +5V -> Net-(LED3-Pad1)
- D21 pad 1: +5V -> Net-(LED3-Pad1)
- D23 pad 1: +5V -> Net-(LED3-Pad1)
- D25 pad 1: +5V -> Net-(LED4-Pad1)
- D25 pad 2: Net-(D25-Pad2) -> Net-(M4O1-Pad2)
- D26 pad 1: Net-(D25-Pad2) -> Net-(M4O1-Pad2)
- D27 pad 1: Net-(C5-Pad2) -> Net-(LED4-Pad1)
- D27 pad 2: Net-(D27-Pad2) -> Net-(M4O1-Pad1)
- D28 pad 1: Net-(C6-Pad2) -> Net-(M4O1-Pad1)
- D28 pad 2: Net-(D28-Pad2) -> GND
- D29 pad 1: +5V -> Net-(LED4-Pad1)
- D29 pad 2: Net-(D29-Pad2) -> Net-(M4O2-Pad2)
- D3 pad 1: +5V -> Net-(C2-Pad1)
- D30 pad 1: Net-(D29-Pad2) -> Net-(M4O2-Pad2)
- D31 pad 1: +5V -> Net-(LED4-Pad1)
- D31 pad 2: Net-(D31-Pad2) -> Net-(M4O2-Pad1)
- D32 pad 1: Net-(D31-Pad2) -> Net-(M4O2-Pad1)
- D5 pad 1: +5V -> Net-(C2-Pad1)
- D7 pad 1: +5V -> Net-(C2-Pad1)
- D9 pad 1: Net-(C1-Pad2) -> Net-(U2-Pad6)
- D9 pad 2: Net-(D9-Pad2) -> Net-(U2-Pad4)
- F1 pad 2: Net-(F1-Pad2) -> Net-(U1-Pad12)
- F2 pad 2: Net-(F2-Pad2) -> Net-(U2-Pad12)
- R1 pad 2: Net-(D9-Pad2) -> Net-(LED1-Pad2)
- R2 pad 2: Net-(D10-Pad2) -> Net-(R2-Pad2)
- R3 pad 2: Net-(D27-Pad2) -> Net-(R3-Pad2)
- R4 pad 2: Net-(D28-Pad2) -> Net-(R4-Pad2)
- U1 pad 12: Net-(F1-Pad2) -> Net-(U1-Pad12)
- U1 pad 6: Net-(C1-Pad2) -> Net-(C2-Pad1)
- U2 pad 2: +3V3 -> GND
- U2 pad 3: CE -> unconnected-(U2-Pad3)
- U2 pad 4: CSN -> Net-(U2-Pad4)
- U2 pad 5: SCK -> Net-(U2-Pad5)
- U2 pad 6: MOSI -> Net-(U2-Pad6)
- U2 pad 7: MISO -> M2 IN1
- U2 pad 8: unconnected-(U2-Pad8) -> M2 PWM1
- U4 pad 12: Net-(F2-Pad2) -> Net-(F4-Pad2)
- U4 pad 13: M3 IN3 -> M4 IN3
- U4 pad 14: M3 PWM2 -> M4 PWM2
- U4 pad 15: M3 IN4 -> M4 IN4
- U4 pad 16: Net-(D13-Pad2) -> Net-(M4O2-Pad2)
- U4 pad 17: Net-(D17-Pad2) -> Net-(M4O2-Pad1)
- U4 pad 4: Net-(D3-Pad2) (its old number) -> Net-(M4O1-Pad2)
- U4 pad 5: Net-(D7-Pad2) (its old number) -> Net-(M4O1-Pad1)
- U4 pad 6: Net-(C2-Pad2) -> Net-(LED4-Pad1)
- U4 pad 7: M3 IN1 -> M4 IN1
- U4 pad 8: M3 PWM1 -> M4 PWM1
- U4 pad 9: M3 IN2 -> M4 IN2
- U5 pad 1: Net-(F1-Pad2) -> +12V
- U6 pad 1: Net-(F2-Pad2) -> GND
- U6 pad 2: GND -> +3V3
- U6 pad 3: +5V -> CE
Routing:
- net Net-(C2-Pad1): track 0.00 -> 107.8 mm
- net GND: track 224.2 -> 117.6 mm, vias 5 -> 4
- net +5V: track 95.9 -> 6.34 mm
- net Net-(D7-Pad2): track 17.3 -> 56.7 mm
- net Net-(D1-Pad2): track 17.3 -> 55.9 mm
- net Net-(C1-Pad2): track 32.3 -> 0.00 mm
- net Net-(D5-Pad2): track 26.5 -> 51.7 mm
- net Net-(D3-Pad2): track 26.5 -> 50.7 mm
- net M1 IN1: track 34.6 -> 11.3 mm, vias 2 -> 0
- net M1 PWM1: track 31.5 -> 9.57 mm, vias 2 -> 0
- net M1 IN2: track 29.0 -> 7.53 mm, vias 2 -> 0
- net Net-(F1-Pad2): track 20.7 -> 0.00 mm
- net Net-(U1-Pad12): track 0.00 -> 16.0 mm
- net Net-(LED1-Pad2): track 0.00 -> 5.26 mm
- net Net-(D9-Pad2): track 5.14 -> 0.00 mm
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- removed copper zone on F.Cu, net +5V
- removed copper zone on B.Cu, net GND

Commit message: progress
Parts:
- added M4O1: PCB_Mounted_XT30, teensy:RightAngleXT30-M, F.Cu at (196.8, 80.2)
- moved LED2 231.3 mm to (123.0, 226.0), turned to 180 degrees
- moved M2O1 214.6 mm to (116.0, 196.8)
- moved D12 214.6 mm to (132.0, 217.5), turned to 180 degrees
- moved C3 212.0 mm to (129.5, 227.5), turned to 90 degrees
- moved D10 198.4 mm to (132.0, 209.5), turned to 180 degrees
- moved D16 196.8 mm to (157.0, 209.5)
- moved D9 182.5 mm to (124.4, 206.0)
- moved D13 170.4 mm to (164.6, 214.2), turned to 180 degrees
- moved D14 167.2 mm to (157.0, 217.8)
- moved C4 159.2 mm to (144.5, 197.5), turned to -90 degrees
- moved R2 151.4 mm to (133.2, 232.0), turned to 180 degrees
- moved C9 145.7 mm to (123.7, 87.0)
- moved D15 138.2 mm to (164.6, 206.0), turned to 180 degrees
- moved D11 134.7 mm to (124.4, 214.0)
- moved U2 131.8 mm to (144.5, 213.0)
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Connections:
- U7 pad 10: M4 IN3 -> M2 IN3
- U7 pad 11: M4 IN4 -> M2 IN2
- U7 pad 12: unconnected-(U7-Pad12) -> M2 PWM1
- U7 pad 16: unconnected-(U7-Pad16) -> M2 IN1
- U7 pad 2: unconnected-(U7-Pad2) -> M1 IN4
- U7 pad 28: M4 PWM2 -> M4 IN4
- U7 pad 29: M4 PWM1 -> M4 PWM2
- U7 pad 3: unconnected-(U7-Pad3) -> M1 PWM2
- U7 pad 30: M2 IN4 -> unconnected-(U7-Pad30)
- U7 pad 31: M2 IN3 -> unconnected-(U7-Pad31)
- U7 pad 32: M2 IN2 -> unconnected-(U7-Pad32)
- U7 pad 33: M2 IN1 -> M4 IN3
- U7 pad 36: M3 PWM2 -> M4 IN2
- U7 pad 37: M3 PWM1 -> M4 PWM1
- U7 pad 38: M1 IN4 -> unconnected-(U7-Pad38)
- U7 pad 39: M1 IN3 -> M4 IN1
- U7 pad 4: M3 IN1 -> M1 IN3
- U7 pad 40: M2 PWM2 -> M3 IN4
- U7 pad 41: M2 PWM1 -> M3 PWM2
- U7 pad 42: M1 IN2 -> M3 IN3
- U7 pad 43: M1 IN1 -> M3 IN2
- U7 pad 44: M1 PWM2 -> M3 PWM1
- U7 pad 45: M1 PWM1 -> M3 IN1
- U7 pad 5: M3 IN2 -> M1 IN2
- U7 pad 6: M3 IN3 -> M1 PWM1
- U7 pad 7: M3 IN4 -> M1 IN1
- U7 pad 8: M4 IN1 -> M2 IN4
- U7 pad 9: M4 IN2 -> M2 PWM2
Routing:
- net GND: track 117.6 -> 377.7 mm, vias 4 -> 8
- net Net-(C3-Pad2): track 0.00 -> 108.9 mm, vias 0 -> 2
- net Net-(C1-Pad2): track 107.8 -> 211.9 mm
- net Net-(D7-Pad2): track 56.7 -> 113.5 mm
- net Net-(D15-Pad2): track 0.00 -> 56.7 mm
- net Net-(D10-Pad1): track 0.00 -> 55.9 mm
- net Net-(D1-Pad2): track 55.9 -> 111.8 mm
- net Net-(D5-Pad2): track 51.7 -> 103.4 mm
- net Net-(D13-Pad2): track 0.00 -> 51.7 mm
- net Net-(D11-Pad2): track 0.00 -> 50.7 mm
- net Net-(D3-Pad2): track 50.7 -> 101.5 mm
- net +5V: track 6.34 -> 23.4 mm
- net M2 IN4: track 0.00 -> 11.5 mm
- net M1 IN4: track 11.5 -> 22.9 mm
- net M2 IN1: track 0.00 -> 11.3 mm
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
Commit message: encoder pins
Parts:
- added A1: Abs Encoder 1, Connector_PinHeader_1.00mm:PinHeader_1x03_P1.00mm_Vertical, F.Cu at (72.5, 228.5)
- added A2: Abs Encoder 2, Connector_PinHeader_1.00mm:PinHeader_1x03_P1.00mm_Vertical, F.Cu at (65.8, 234.6)
- added A3: Abs Encoder 3, Connector_PinHeader_1.00mm:PinHeader_1x03_P1.00mm_Vertical, F.Cu at (72.5, 233.6)
- added A4: Abs Encoder 4, Connector_PinHeader_1.00mm:PinHeader_1x03_P1.00mm_Vertical, F.Cu at (78.3, 228.5)
- added Q1: Quad Encoder 1, Connector_PinHeader_1.00mm:PinHeader_1x04_P1.00mm_Vertical, F.Cu at (69.3, 228.5)
- added Q2: Quad Encoder 2, Connector_PinHeader_1.00mm:PinHeader_1x04_P1.00mm_Vertical, F.Cu at (62.6, 234.6)
- added Q3: Quad Encoder 3, Connector_PinHeader_1.00mm:PinHeader_1x04_P1.00mm_Vertical, F.Cu at (66.0, 228.5)
- added Q4: Quad Encoder 4, Connector_PinHeader_1.00mm:PinHeader_1x04_P1.00mm_Vertical, F.Cu at (62.6, 228.5)
- moved D14 34.9 mm to (191.7, 222.0)
- moved D15 34.9 mm to (199.3, 210.2)
- moved D16 34.9 mm to (191.7, 213.8)
- moved D13 34.8 mm to (199.3, 217.5)
- moved M1O1 23.0 mm to (63.5, 18.5)
- moved M1O2 22.9 mm to (77.5, 18.5)
Connections:
- D5 pad 2: Net-(D5-Pad2) -> Net-(D6-Pad1)
- D6 pad 1: Net-(D5-Pad2) -> Net-(D6-Pad1)
- D7 pad 2: Net-(D7-Pad2) -> Net-(D8-Pad1)
- D8 pad 1: Net-(D7-Pad2) -> Net-(D8-Pad1)
- M1O2 pad 1: Net-(D7-Pad2) -> Net-(D6-Pad1)
- M1O2 pad 2: Net-(D5-Pad2) -> Net-(D8-Pad1)
- M2O2 pad 1: Net-(D15-Pad2) -> Net-(D13-Pad2)
- M2O2 pad 2: Net-(D13-Pad2) -> Net-(D15-Pad2)
- M3O2 pad 1: Net-(D23-Pad2) -> Net-(D21-Pad2)
- M3O2 pad 2: Net-(D21-Pad2) -> Net-(D23-Pad2)
- M4O2 pad 1: Net-(D31-Pad2) -> Net-(D29-Pad2)
- M4O2 pad 2: Net-(D29-Pad2) -> Net-(D31-Pad2)
- U1 pad 16: Net-(D5-Pad2) -> Net-(D8-Pad1)
- U1 pad 17: Net-(D7-Pad2) -> Net-(D6-Pad1)
- U2 pad 16: Net-(D13-Pad2) -> Net-(D15-Pad2)
- U2 pad 17: Net-(D15-Pad2) -> Net-(D13-Pad2)
- U3 pad 16: Net-(D21-Pad2) -> Net-(D23-Pad2)
- U3 pad 17: Net-(D23-Pad2) -> Net-(D21-Pad2)
- U4 pad 16: Net-(D29-Pad2) -> Net-(D31-Pad2)
- U4 pad 17: Net-(D31-Pad2) -> Net-(D29-Pad2)
Routing:
- net Net-(D7-Pad2): track 113.5 -> 0.00 mm
- net (no net): track 0.00 -> 108.5 mm
- net Net-(D5-Pad2): track 103.4 -> 0.00 mm
- net Net-(D6-Pad1): track 0.00 -> 74.9 mm
- net Net-(D8-Pad1): track 0.00 -> 69.3 mm
- net Net-(C3-Pad2): track 108.9 -> 67.9 mm, vias 2 -> 0
- net Net-(D1-Pad2): track 111.8 -> 130.8 mm
- net Net-(D3-Pad2): track 101.5 -> 119.9 mm
- net GND: track 377.7 -> 364.1 mm
- net Net-(D15-Pad2): track 56.7 -> 51.7 mm
- net Net-(D13-Pad2): track 51.7 -> 56.7 mm
