File: swervepcb.kicad_sch (KiCad schematic)
At the start: 74 parts, among them J1 RJ45_LED, U1 Teensy4.1, U10 PCB_Mounted_XT30, U11 BAT, U12 L298P, U13 L298P, U14 L7805, U15 L7805, U16 PCB_Mounted_XT30, U17 PCB_Mounted_XT30, U18 PCB_Mounted_XT30, U19 PCB_Mounted_XT30, U2 NRF24L01_Breakout, U3 L298P, U4 L298P, U5 L7805, U6 L7805, U7 PCB_Mounted_XT30, U8 PCB_Mounted_XT30, U9 PCB_Mounted_XT30

Commit message: progress
Parts:
- removed C2: 220uF, Capacitor_THT:CP_Radial_D8.0mm_P3.50mm, symbol Device:C_Small
- removed D10, D27, D28, D9: PWR-LED, LED_THT:LED_D5.0mm, symbol Device:LED
- removed D3, D33, D34, D35, D36, D4, D7, D8: (no value), Diode_THT:D_DO-41_SOD81_P7.62mm_Horizontal, symbol Device:D_Small
- removed F5: 2a, Fuse:Fuseholder_Cylinder-5x20mm_Schurter_0031_8201_Horizontal_Open, symbol Device:Fuse_Small
- removed U10, U16, U17, U18, U19, U9: PCB_Mounted_XT30, teensy:RightAngleXT30-M, symbol xt30:PCB_Mounted_XT30
- removed U12, U13: L298P, L298P:L298P, symbol Driver_Motor:L298P
- removed U14, U15, U6: L7805, L7805CV:STMicroelectronics-TO-220-3-0-0-0, symbol Regulator_Linear:L7805
- added C3: 220uF, Capacitor_THT:CP_Radial_D8.0mm_P3.50mm, symbol Device:C_Small
- added D10, D11, D12, D15, D16, D27, D28, D9: (no value), Diode_THT:D_DO-41_SOD81_P7.62mm_Horizontal, symbol Device:D_Small
- added F3: 2a, Fuse:Fuseholder_Cylinder-5x20mm_Schurter_0031_8201_Horizontal_Open, symbol Device:Fuse_Small
- added LED1, LED2, LED3, LED4: PWR-LED, LED_THT:LED_D5.0mm, symbol Device:LED
- added M2O1, M2O2, M3O1, M3O2, M4O1, M4O2: PCB_Mounted_XT30, teensy:RightAngleXT30-M, symbol xt30:PCB_Mounted_XT30
- added U2, U3: L298P, L298P:L298P, symbol Driver_Motor:L298P
- C8: footprint Diode_THT:D_DO-41_SOD81_P7.62mm_Horizontal -> Capacitor_THT:CP_Radial_D8.0mm_P3.50mm
- F0: renamed from F3; value 10a -> 8a
- R1, R2, R3, R4: footprint Resistor_SMD:R_0805_2012Metric_Pad1.20x1.40mm_HandSolder -> Resistor_THT:R_Axial_DIN0309_L9.0mm_D3.2mm_P12.70mm_Horizontal
- renumbered C3 to C2, D5 to D3, D6 to D4, D11 to D5, D12 to D6, D15 to D7, D16 to D8, U7 to M1O1, U8 to M1O2, U11 to U0, U3 to U1, U2 to U6, U1 to U7
Connections:
- net +12V: now also U5.1 (IN), F3.1
- net +5V: now also C3.1; no longer C2.1, C4.1, C6.1, C8.1, D1.1 (K), D13.1 (K), D17.1 (K), D19.1 (K), D21.1 (K), D23.1 (K), D25.1 (K), D29.1 (K), D3.1 (K), D31.1 (K), D5.1 (K), D7.1 (K)
- net GND: now also C6.2, D10.2 (A), D12.2 (A), D16.2 (A), D28.2 (A), U2.1 (GND), U2.10 (GND), U2.11 (GND), U2.19 (SENSE_B), U2.2 (SENSE_A), U2.20 (GND), U3.1 (GND), U3.10 (GND), U3.11 (GND), U3.19 (SENSE_B), U3.2 (SENSE_A), U3.20 (GND); no longer C7.2
- net M2 IN1: now also U2.7 (IN1)
- net M2 IN2: now also U2.9 (IN2)
- net M2 IN3: now also U2.13 (IN3)
- net M2 IN4: now also U2.15 (IN4)
- net M2 PWM1: now also U2.8 (EnA)
- net M2 PWM2: now also U2.14 (EnB)
- net M3 IN1: now also U3.7 (IN1); no longer U4.7 (IN1)
- net M3 IN2: now also U3.9 (IN2); no longer U4.9 (IN2)
- net M3 IN3: now also U3.13 (IN3); no longer U4.13 (IN3)
- net M3 IN4: now also U3.15 (IN4); no longer U4.15 (IN4)
- net M3 PWM1: now also U3.8 (EnA); no longer U4.8 (EnA)
- net M3 PWM2: now also U3.14 (EnB); no longer U4.14 (EnB)
- net M4 IN1: now also U4.7 (IN1)
- net M4 IN2: now also U4.9 (IN2)
- net M4 IN3: now also U4.13 (IN3)
- net M4 IN4: now also U4.15 (IN4)
- net M4 PWM1: now also U4.8 (EnA)
- net M4 PWM2: now also U4.14 (EnB)
- net at D13.2 (A), D14.1 (K): now also M2O2.2, U2.16 (OUT3); no longer U4.16 (OUT3)
- net at C5.2: now also C6.1, D17.1 (K), D19.1 (K), D21.1 (K), D23.1 (K), LED3.1 (K), U3.6 (Vs)
- net at F2.2: now also U2.12 (Vss); no longer U4.12 (Vss)
- net at D17.2 (A), D18.1 (K): now also M3O1.2, U3.4 (OUT1); no longer U4.17 (OUT4)
- net at U4.4 (OUT1): now also D25.2 (A), D26.1 (K), M4O1.2
- net at U4.5 (OUT2): now also D27.2 (A), D28.1 (K), M4O1.1
- net at U4.6 (Vs): now also C7.2, C8.1, D25.1 (K), D29.1 (K), D31.1 (K), D27.1 (K), LED4.1 (K)
- net at D31.2 (A), D32.1 (K): now also U4.17 (OUT4), M4O2.1
- net at R4.2: now also LED4.2 (A)
- net at D19.2 (A), D20.1 (K): now also M3O1.1, U3.5 (OUT2)
- net at D21.2 (A), D22.1 (K): now also M3O2.2, U3.16 (OUT3)
- net at C1.2, U1.6 (Vs): now also C2.1, D1.1 (K), D3.1 (K), D5.1 (K), D7.1 (K), LED1.1 (K)
- net at R2.2: now also LED2.2 (A)
- net at F4.2: now also U4.12 (Vss)
- net at D29.2 (A), D30.1 (K): now also U4.16 (OUT3), M4O2.2
- net at D23.2 (A), D24.1 (K): now also M3O2.1, U3.17 (OUT4)
- net at R1.2: now also LED1.2 (A)
- net at F1.2, U1.12 (Vss): no longer U5.1 (IN)
- net at R3.2: now also LED3.2 (A)
- new net: D15.2 (A), D16.1 (K), M2O2.1, U2.17 (OUT4)
- new net: D10.1 (K), D9.2 (A), M2O1.2, U2.4 (OUT1)
- new net: D11.2 (A), D12.1 (K), M2O1.1, U2.5 (OUT2)
- new net: C3.2, C4.1, D11.1 (K), D13.1 (K), D15.1 (K), D9.1 (K), LED2.1 (K), U2.6 (Vs)
- new net: F3.2, U3.12 (Vss)
Other:
- moved on the sheet: C2, F0, F1, U0, U5

Commit message: progress
Connections:
- net M1 IN1: now also U7.7 (5_IN2); no longer U7.43 (21_A7_RX5_BCLK1)
- net M1 IN2: now also U7.5 (3_LRCLK2); no longer U7.42 (20_A6_TX5_LRCLK1)
- net M1 IN3: now also U7.4 (2_OUT2); no longer U7.39 (17_A3_TX4_SDA1)
- net M1 IN4: now also U7.2 (0_RX1_CRX2_CS1); no longer U7.38 (16_A2_RX4_SCL1)
- net M1 PWM1: now also U7.6 (4_BCLK2); no longer U7.45 (23_A9_CRX1_MCLK1)
- net M1 PWM2: now also U7.3 (1_TX1_CTX2_MISO1); no longer U7.44 (22_A8_CTX1)
- net M2 IN1: now also U7.16 (24_A10_TX6_SCL2); no longer U7.33 (41_A17)
- net M2 IN2: now also U7.11 (9_OUT1C); no longer U7.32 (40_A16)
- net M2 IN3: now also U7.10 (8_TX2_IN1); no longer U7.31 (39_MISO1_OUT1A)
- net M2 IN4: now also U7.8 (6_OUT1D); no longer U7.30 (38_CS1_IN1)
- net M2 PWM1: now also U7.12 (10_CS_MQSR); no longer U7.41 (19_A5_SCL)
- net M2 PWM2: now also U7.9 (7_RX2_OUT1A); no longer U7.40 (18_A4_SDA)
- net M3 IN1: now also U7.45 (23_A9_CRX1_MCLK1); no longer U7.4 (2_OUT2)
- net M3 IN2: now also U7.43 (21_A7_RX5_BCLK1); no longer U7.5 (3_LRCLK2)
- net M3 IN3: now also U7.42 (20_A6_TX5_LRCLK1); no longer U7.6 (4_BCLK2)
- net M3 IN4: now also U7.40 (18_A4_SDA); no longer U7.7 (5_IN2)
- net M3 PWM1: now also U7.44 (22_A8_CTX1); no longer U7.37 (15_A1_RX3_SPDIF_IN)
- net M3 PWM2: now also U7.41 (19_A5_SCL); no longer U7.36 (14_A0_TX3_SPDIF_OUT)
- net M4 IN1: now also U7.39 (17_A3_TX4_SDA1); no longer U7.8 (6_OUT1D)
- net M4 IN2: now also U7.36 (14_A0_TX3_SPDIF_OUT); no longer U7.9 (7_RX2_OUT1A)
- net M4 IN3: now also U7.33 (41_A17); no longer U7.10 (8_TX2_IN1)
- net M4 IN4: now also U7.28 (36_CS); no longer U7.11 (9_OUT1C)
- net M4 PWM1: now also U7.37 (15_A1_RX3_SPDIF_IN); no longer U7.29 (37_CS)
- net M4 PWM2: now also U7.29 (37_CS); no longer U7.28 (36_CS)

Commit message: encoder pins
Parts:
- added A1: Abs Encoder 1, Connector_PinHeader_1.00mm:PinHeader_1x03_P1.00mm_Vertical, symbol Connector:Conn_01x03_Female
- added A2: Abs Encoder 2, Connector_PinHeader_1.00mm:PinHeader_1x03_P1.00mm_Vertical, symbol Connector:Conn_01x03_Female
- added A3: Abs Encoder 3, Connector_PinHeader_1.00mm:PinHeader_1x03_P1.00mm_Vertical, symbol Connector:Conn_01x03_Female
- added A4: Abs Encoder 4, Connector_PinHeader_1.00mm:PinHeader_1x03_P1.00mm_Vertical, symbol Connector:Conn_01x03_Female
- added Q1: Quad Encoder 1, Connector_PinHeader_1.00mm:PinHeader_1x04_P1.00mm_Vertical, symbol Connector:Conn_01x04_Female
- added Q2: Quad Encoder 2, Connector_PinHeader_1.00mm:PinHeader_1x04_P1.00mm_Vertical, symbol Connector:Conn_01x04_Female
- added Q3: Quad Encoder 3, Connector_PinHeader_1.00mm:PinHeader_1x04_P1.00mm_Vertical, symbol Connector:Conn_01x04_Female
- added Q4: Quad Encoder 4, Connector_PinHeader_1.00mm:PinHeader_1x04_P1.00mm_Vertical, symbol Connector:Conn_01x04_Female
- renumbered D7 to D5, D8 to D6, D5 to D7, D6 to D8
Connections:
- net +5V: now also A1.1 (Pin_1), A2.1 (Pin_1), A3.1 (Pin_1), A4.1 (Pin_1), Q1.2 (Pin_2), Q2.2 (Pin_2), Q3.2 (Pin_2), Q4.2 (Pin_2)
- net GND: now also A1.3 (Pin_3), A2.3 (Pin_3), A3.3 (Pin_3), A4.3 (Pin_3), Q1.4 (Pin_4), Q2.4 (Pin_4), Q3.4 (Pin_4), Q4.4 (Pin_4)
- net at D31.2 (A), D32.1 (K): now also M4O2.2, U4.16 (OUT3); no longer M4O2.1, U4.17 (OUT4)
- net at D13.2 (A), D14.1 (K): now also M2O2.1, U2.17 (OUT4); no longer M2O2.2, U2.16 (OUT3)
- net at D23.2 (A), D24.1 (K): now also M3O2.2, U3.16 (OUT3); no longer M3O2.1, U3.17 (OUT4)
- net at D29.2 (A), D30.1 (K): now also M4O2.1, U4.17 (OUT4); no longer M4O2.2, U4.16 (OUT3)
- net at D15.2 (A), D16.1 (K): now also M2O2.2, U2.16 (OUT3); no longer M2O2.1, U2.17 (OUT4)
- net at D21.2 (A), D22.1 (K): now also M3O2.1, U3.17 (OUT4); no longer M3O2.2, U3.16 (OUT3)
- new net A1S: A1.2 (Pin_2)
- new net A2S: A2.2 (Pin_2)
- new net A3S: A3.2 (Pin_2)
- new net A4S: A4.2 (Pin_2)
- new net Q1A: Q1.3 (Pin_3)
- new net Q1B: Q1.1 (Pin_1)
- new net Q2A: Q2.3 (Pin_3)
- new net Q2B: Q2.1 (Pin_1)
- new net Q3A: Q3.3 (Pin_3)
- new net Q3B: Q3.1 (Pin_1)
- new net Q4A: Q4.3 (Pin_3)
- new net Q4B: Q4.1 (Pin_1)
Other:
- moved on the sheet: C9, D13, D14, D15, D16, D21, D22, D23, D24, D29, D30, D31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
